File: Hardware/PQ60-EPS.sch (EAGLE design)
At the start: 23 parts, among them IC1 LTC4413, IC3 MKL05Z32VFM4, J1 FTS-105-01-L-D, X1-BOT FX8C-60S-SV, X1-TOP FX8C-60P-SV, X5 M02SMD

Commit message: Broken out some modules. Swapping SMPS.
Parts:
- added C10, C13, C15, C8: 10uF, rcl:C-EUC0603
- added C11, C16, C18: 4.7uF, rcl:C-EUC0603
- added C12, C17: 10nF, rcl:C-EUC0603
- added C14, C9: 1uF, rcl:C-EUC0603
- added C19: 100nF, rcl:C-EUC0603
- added IC2, IC5: LTC3105, general:LTC3105EMSPBF
- added IC6: MAX8606, general:MAX8606ETD+T
- added L1, L2: 10uH, WE-TPC:WE-TPC-744031100_3816
- added R10, R8, R9: 2k, rcl:R-EU_R0603
- added R2, R5: 75k, rcl:R-EU_R0603
- added R3, R6: 1M33, rcl:R-EU_R0603
- added R4, R7: 392k, rcl:R-EU_R0603
- added U$1: TPS630250, ears-pq:TPS630250
- added U$2: XAL4020, ears-pq:XAL4020
Connections:
- new net !SHDN1!: IC2.!SHDN!
- new net !SHDN2!: IC5.!SHDN!
- new net AUX1: C9.1, IC2.AUX
- new net AUX2: C14.1, IC5.AUX
- new net FB1: IC2.FB, R3.1, R4.2
- new net FB2: IC5.FB, R6.1, R7.2
- new net IN: IC5.V+, IC5.VIN-, R5.2, R7.1
- new net I_LIM_SW1: IC2.ILIM, R2.1
- new net I_SEN: IC5.OUT, R6.1
- new net LDO1: C11.2, IC2.LDO
- new net LDO2: C16.2, IC5.LDO
- new net MPPC1: IC2.MPPC, R2.2
- new net MPPC2: IC5.MPPC, R5.2
- new net N$6: U$1.L1, U$2.P$1
- new net N$7: U$1.L2, U$2.P$2
- new net N$9: R10.2, R9.1, U$1.FB
- new net OUT_SW1: IC2.OUT
- new net SW1: IC2.SW, L1.2
- new net SW1_!FAULT!: IC2.~FAULT
- new net SW1_EN: IC2.EN
- new net SW2: IC5.SW, L2.2
- new net THM1: C12.1, R2.1
- new net THM2: C17.1, R5.1
- new net V_SEN: R7.2, R8.1
- net +3V3_UNPRO: now also R9.2
- net BATT_PROG: now also IC6.SETI, R8.2
- net BMS_!CHG!: now also IC6.~CHG
- net BMS_!PGD!: now also IC6.~POK
- net FB: now also R2.1, R3.2
- net GND: now also C10.2, C11.1, C12.2, C13.2, C14.2, C15.2, C16.1, C17.2, C18.1, C19.1, C8.2, C9.2, IC2.EP, IC2.FBLDO, IC2.GND, IC2.GND@6, IC2.GND@7, IC5.FBLDO, IC5.GND, IC5.GND@6, IC5.GND@7, IC6.EP, IC6.GND, IC6.~EN1, IC6.~EN2, IC6.~TMR, R10.1, R2.2, R3.1, R3.2, R4.1, R4.2, R6.2, R7.1, R8.1, R8.2, U$1.GND, U$1.PFM/PWM, U$1.PGND
- net IN_SEN: now also IC2.IN, IC5.VIN+, R5.1
- net I_LIM_SW2: now also R3.1
- net I_LIM_SW3: now also R4.1
- net MPPT_PGD: now also IC2.PGOOD
- net N$1: now also L1.1
- net N$2: now also L1.2
- net PGOOD: now also IC5.PGOOD
- net SOLAR[1..2]: now also C8.1, IC2.VIN, L1.1
- net SOLAR[3..4]: now also C13.1, IC5.VIN, L2.1
- net SW: now also L1.2
- net S_ARRAY_1: now also C10.1, IC2.VOUT, R3.2
- net S_ARRAY_2: now also C15.1, IC5.VOUT, R6.2
- net THM: now also IC6.THM
- net VIN: now also L1.1
- net VL: now also C19.2, IC6.VL
- net VOUT: now also R2.2
- net VSOL: now also C18.2, IC6.IN
- net VSYS: now also IC6.SYS@1, IC6.SYS@2
- net VSYS_SW: now also U$1.EN, U$1.VIN, U$1.VINA
- net V_BAT: now also IC6.BAT@1, IC6.BAT@2
Other:
- moved on the sheet: C4, IC1, X2, X3, X4, X5

Commit message: pre deleting prot modules
Parts:
- removed R10, R9: 2k, rcl:R-EU_R0603
- added C20, C21: 10uF, rcl:C-EUC0603
- added U$3, U$5, U$6: INA3221, ears-pq:INA3221
- added U$4, U$7, U$8, U$9: TPS2052B, ears-pq:TPS2052B
Connections:
- net N$6 renamed L1
- net N$7 renamed L2
- new net 3V3_PRO: U$6.VINI2-
- new net N$10: U$5.VIN2+, U$8.OUT2
- new net N$11: U$5.VIN3+, U$9.OUT1
- new net N$12: U$6.VIN1+, U$9.OUT2
- new net N$13: U$6.VIN2+, U$7.OUT2
- new net N$6: U$3.VIN1+, U$4.OUT1
- new net N$7: U$3.VIN2+, U$4.OUT2
- new net N$8: U$3.VIN3+, U$7.OUT1
- net +3V3_SW[1]: now also U$3.VIN1-
- net +3V3_SW[2]: now also U$3.VINI2-
- net +3V3_SW[3]: now also U$3.VIN3-
- net +3V3_UNPRO: now also C21.1, U$1.FB, U$1.VOUT, U$4.IN, U$7.IN; no longer R9.2
- net GND: now also C20.2, C21.2, U$3.A0, U$3.GND, U$4.GND, U$5.GND, U$6.GND, U$7.GND, U$8.GND, U$9.GND; no longer R10.1
- net I2C_SCL: now also U$3.SCL, U$5.A0, U$5.SCL, U$6.SCL
- net I2C_SDA: now also U$3.SDA, U$5.SDA, U$6.A0, U$6.SDA
- net N$9: now also U$5.VIN1+, U$8.OUT1; no longer R10.2, R9.1, U$1.FB
- net VBAT: now also U$6.VIN1-
- net VBAT_SW[1]: now also U$5.VIN1-
- net VBAT_SW[1]_EN: now also U$8.!EN1!
- net VBAT_SW[2]: now also U$5.VINI2-
- net VBAT_SW[2]_EN: now also U$8.!EN2!
- net VBAT_SW[3]: now also U$5.VIN3-
- net VBAT_SW[3]_EN: now also U$9.!EN1!
- net VSYS_SW: now also C20.1, U$3.VS, U$5.VS, U$6.VS, U$8.IN, U$9.!EN2!, U$9.IN
Other:
- moved on the sheet: U$1, U$2

Commit message: routed most of the power
Parts:
- removed C7: 100nF, rcl:C-EUC0603
- removed IC3: MKL05Z32VFM4, general:MKL05Z32VFM4
- removed J1: FTS-105-01-L-D, general:FTS-105-01-L-D
- removed R16: DNP, rcl:R-EU_R0603
- removed TP1: TEST-POINT2, SparkFun-Passives:TEST-POINT2
- removed TP2: TEST-POINT3, SparkFun-Passives:TEST-POINT3
- added R10, R11, R12, R13, R14, R9: 1M33, rcl:R-EU_R0603
- R1: value 10k -> 1M33
- R15: value DNP -> 1M33
Connections:
- removed net +3V3_I_SEN: IC3.PTB2/IRQ_10/LLWU_P5
- removed net +3V3_SW[0]_!FAULT!: IC3.PTB11
- removed net +3V3_SW[1]_!FAULT!: IC3.PTB10
- removed net +3V3_SW[1]_EN: IC3.PTB9
- removed net +3V3_SW[2]_!FAULT!: IC3.PTB8
- removed net +3V3_SW[2]_EN: IC3.PTA6/LLWU_P2
- removed net +3V3_SW[3]_!FAULT!: IC3.PTA5/LLWU_P1/RTC_CLK_IN
- removed net +3V3_SW[3]_EN: IC3.PTA4/LLWU_P0
- removed net +3V3_V_SEN: IC3.PTA8
- removed net I2C_INT: IC3.PTB5/IRQ_16, TP2.1
- removed net N$5: IC3.VREFH, TP1.1
- removed net OUT_SW2: IC3.OUT
- removed net PRO1: C1.1, IC4.VCC, R15.2, R16.2, X1-BOT.+3V3@57, X1-BOT.+3V3@58, X1-BOT.+3V3@59, X1-BOT.+3V3@60, X1-TOP.+3V3@57, X1-TOP.+3V3@58, X1-TOP.+3V3@59, X1-TOP.+3V3@60
- removed net RESET: IC3.PTA1/IRQ_1/LPTMR0_ALT1, J1.!RESET, R1.1
- removed net SW2_!FAULT!: IC3.~FAULT
- removed net SW2_EN: IC3.EN
- removed net SWD_CLK: IC3.PTA0/IRQ_0/LLWU_P7, J1.SWDCLK/TCK
- removed net SWD_DIO: IC3.PTA2, J1.SWDIO/TMS
- removed net VBAT_I_SEN: IC3.PTB0/IRQ_8/LLWU_P4
- removed net VBAT_SW[0]_!FAULT!: IC3.PTA7/IRQ_7/LLWU_P3
- removed net VBAT_SW[1]_!FAULT!: IC3.PTA13
- removed net VBAT_SW[2]_!FAULT!: IC3.PTB12
- removed net VBAT_SW[3]_!FAULT!: IC3.PTB13
- removed net VBAT_V_SEN: IC3.PTB1/IRQ_9
- net +3V3_SW[1]: now also R1.1
- net +3V3_SW[2]: now also R9.1
- net +3V3_SW[3]: now also R10.1
- net +3V3_UNPRO: now also U$7.!EN2!; no longer C7.1, IC3.VDD, J1.VCC, R1.2
- net 3V3_PRO: now also C1.1, IC4.VCC, R15.1, U$6.VIN1-, X1-BOT.+3V3@57, X1-BOT.+3V3@58, X1-BOT.+3V3@59, X1-BOT.+3V3@60, X1-TOP.+3V3@57, X1-TOP.+3V3@58, X1-TOP.+3V3@59, X1-TOP.+3V3@60; no longer U$6.VINI2-
- net BMS_!CHG!: no longer IC3.PTA10/IRQ_12
- net BMS_!PGD!: no longer IC3.PTA9
- net GND: no longer C7.2, IC3.EP, IC3.GND, IC3.THERMAL_PAD, IC3.VREFL, IC3.VSS, J1.GND@3, J1.GND@5, J1.GND_DET, J1.KEY
- net I2C_SCL: no longer IC3.PTB3/IRQ_14, R16.1
- net I2C_SDA: no longer IC3.PTB4/IRQ_15/LLWU_P6, R15.1
- net IDIODE_STAT: no longer IC3.PTA11/IRQ_13
- net IN_SEN: no longer IC3.IN
- net I_LIM_SW2: no longer IC3.ILIM
- net MPPT_PGD: no longer IC3.PTA12/IRQ_17/LPTMR0_ALT2
- net N$10: now also R12.2
- net N$11: now also R13.2
- net N$12: now also R14.2, U$6.VIN3+; no longer U$6.VIN1+
- net N$13: now also R15.2, U$6.VIN1+; no longer U$6.VIN2+
- net N$6: now also R1.2
- net N$7: now also R9.2
- net N$8: now also R10.2
- net N$9: now also R11.2
- net VBAT: now also R14.1, U$6.VIN3-; no longer U$6.VIN1-
- net VBAT_SW[1]: now also R11.1
- net VBAT_SW[1]_EN: no longer IC3.PTA3
- net VBAT_SW[2]: now also R12.1
- net VBAT_SW[2]_EN: no longer IC3.PTB7/IRQ_3
- net VBAT_SW[3]: now also R13.1
- net VBAT_SW[3]_EN: no longer IC3.PTB6/IRQ_2/LPTMR0_ALT3
Other:
- note removed: "sw: I2C/SMBus/PMBus interface 2 output blocks MPPT Status IDiode Status BMS Status SMPS Status"
- moved on the sheet: R1, R15, U$6
